File: kicad/mixer-board/mixer-board.sch (KiCad schematic (older format))
At the start: 25 parts

Commit message: New schematic for the mixer-board with feedback from forum.
Parts:
- removed R? (x12): 100k, SM0603S, symbol R
- added ACC1: ADXL345, symbol ADXL345
- added ACC2: BMA180, symbol BMA180
- added C2: 10uF, symbol CP1
- added C3, C6: 0.22nF, symbol C
- added C4, C5: 0.1uF, symbol C
- added C9: 100nF, symbol C
- added GConn1, GConn2, GConn3, GConn4, GConn5, GConn6: GCONN, symbol GCONN
- added JC1: JEEPORT, symbol JEEPORT
- added R? (x2): 47k, symbol R
- added SJ1, SJ?: SOLDER_JUMPER, symbol SOLDER_JUMPER
- added U1: ADXL345_BREAKOUT_BOARD, symbol ADXL345_BREAKOUT_BOARD
- added U4: TMP36, symbol TMP36
- gave numbers to parts that had none: 13
Connections:
- net labels added: I2C_SCL, I2C_SDA, SENSOR_ENA
- wire segments 111 -> 176
- no-connect marks 5 -> 10
Other:
- note added: "K1"
- note added: "K2"
- note added: "K3"
- note added: "K4"
- note added: "K5"
- note added: "K6"
