File: kicad/usb-board/usb_board.sch (KiCad schematic (older format))
At the start: 24 parts, among them J1 USB_2, P1 CONN_8, P2 CONN_8, P3 CONN_8, SW1 SW_PUSH_SMALL, U1 PANSTAMP_02, U2 FT232RL, U3 MCP1702

Commit message: Grove connectors and fuse
Parts:
- removed P3: CONN_8, SIL-8, symbol CONN_8
- added F1: PTC 500mA, SM0805, symbol FUSE
- added P3, P4: CONN_4, GROVE_MALE, symbol CONN_4
- added R4, R5: 4k7, SM0603S, symbol R
- P1, P2: value CONN_8 -> CONN_12; footprint SIL-8 -> SIL-12; symbol CONN_8 -> CONN_12
Connections:
- net labels added: A4_SDA, A5_SCL
- net labels removed: A4, A5
- wire segments 111 -> 130
