File: kicad/output-board/relays.sch (KiCad schematic (older format))
At the start: 56 parts, among them Q1 NPN, Q2 NPN, Q3 NPN, Q4 NPN, Q5 NPN, Q6 NPN, Q7 NPN, Q8 NPN, U10 SONGLE_RELAY_10A, U3 SONGLE_RELAY_10A, U4 SONGLE_RELAY_10A, U5 SONGLE_RELAY_10A, U6 SONGLE_RELAY_10A, U7 SONGLE_RELAY_10A, U8 SONGLE_RELAY_10A, U9 SONGLE_RELAY_10A

Commit message: New PCB layout in accordance with the CE directives
Parts:
- BIN7: value CONN_3 -> CONN_2; footprint BORNIER3 -> BORNIER2; symbol CONN_3 -> CONN_2
- R10, R11, R12, R13, R2, R3, R4, R5: value 470 -> 1k5
- R14, R15, R16, R17, R6, R7, R8, R9: value 1k -> 2k2
Connections:
- net +12V: now also R10.1, R11.1, R12.1, R13.1, R2.2, R3.1, R4.1, R5.1
- net BINOUT0: no longer R2.2
- net BINOUT1: no longer R3.2
- net BINOUT2: no longer R4.2
- net BINOUT3: no longer R5.2
- net BINOUT4: no longer R10.2
- net BINOUT5: no longer R11.2
- net BINOUT6: no longer R12.2
- net BINOUT7: no longer R13.2
- net GND: no longer D11.2 (K), D12.2 (K), D13.2 (K), D14.2 (K), D3.2 (K), D4.2 (K), D5.2 (K), D6.2 (K)
- net at D7.1 (A), Q1.3 (C), U3.3: now also D3.2 (K)
- net at D8.1 (A), Q2.3 (C), U4.3: now also D4.2 (K)
- net at D4.1 (A): now also R3.2; no longer R3.1
- net at D6.1 (A): now also R5.2; no longer R5.1
- net at D10.1 (A), Q4.3 (C), U6.3: now also D6.2 (K)
- net at D9.1 (A), Q3.3 (C), U5.3: now also D5.2 (K)
- net at D5.1 (A): now also R4.2; no longer R4.1
- net at D13.1 (A): now also R12.2; no longer R12.1
- net at BIN7.1 (P1): now also U9.2; no longer U9.4
- net at BIN7.2 (PM): now also U9.5; no longer U9.2
- net at D17.1 (A), Q7.3 (C), U9.3: now also D13.2 (K)
- net at D18.1 (A), Q8.3 (C), U10.3: now also D14.2 (K)
- net at D14.1 (A): now also R13.2; no longer R13.1
- net at D12.1 (A): now also R11.2; no longer R11.1
- net at D16.1 (A), Q6.3 (C), U8.3: now also D12.2 (K)
- net at D15.1 (A), Q5.3 (C), U7.3: now also D11.2 (K)
- net at D11.1 (A): now also R10.2; no longer R10.1
- no-connect marks 0 -> 1
Other:
- moved on the sheet: BIN1, BIN2, BIN3, BIN4, D10, D11, D12, D13, D14, D3, D4, D5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
