File: kicad/panstamp-nrg/panstamp.sch (KiCad schematic (older format))
At the start: 56 parts, among them P1 CONN_12, P2 CONN_12, P3 CONN_5, U1 CC430F5137, U2 0868BM15C0001, U4 MMA8652FC, U6 BMP085, X1 26MHz

Commit message: New PCB layout
Parts:
- removed R2, R3, R9: 10k, SM0603S, symbol R
- removed U2: 0868BM15C0001, JTI_Balun, symbol BALUN+FILTER
- removed U6: BMP085, BMP085, symbol BMP085
- added C14, C30: 10u, SM0603S, symbol C
- added C7: 100n, SM0402, symbol C
- added U3: SI7021, DFN-6, symbol SI7021
- C1: value 4.7u -> 10u; footprint SM0402 -> SM0603S
- L1, L2: value 12n -> 600R/200mA
- R1: footprint SM0402 -> SM0603
- TH1: footprint SM0402 -> SM0603S
Connections:
- net GND: now also C14.1, C30.2, C7.1, U3.2 (GND)
- net I2C_SCL: now also U3.6 (SCL)
- net I2C_SDA: now also U3.1 (SDA)
- net P2.1/A1: now also R1.1, TH1.1
- net P2.2/A2: now also TH1.2
- net P2.5/A5: now also C30.1; no longer R1.1, TH1.1
- net P3.3: now also U4.1 (VDD)
- net PJ.2: no longer TH1.2
- net VCC: now also U3.5 (Vdd); no longer U4.1 (VDD)
- net at L2.2, U1.45 (AVCC): now also C14.2, C7.2
- no-connect marks 2 -> 0
Other:
- moved on the sheet: C16, C17, C19, C21, L2, LED1, R1, R5, R6, R8, TH1, U4
